Commit message: control bar for test pybullet gym

File: test/hole.urdf (robot description, URDF)
Before this commit: robot hole, 7 links, 6 joints
Links:
- link hole_left: geometry collision box size=0.44 0.1 0.053; visual box size=0.44 0.02 0.053
- link hole_right: geometry collision box size=0.44 0.1 0.053; visual box size=0.44 0.02 0.053

File: test/peg.urdf (robot description, URDF)
Before this commit: robot peg, 5 links, 4 joints
Links:
- link peg: geometry collision box size=0.11 0.02 0.053; visual box size=0.11 0.02 0.053
- link target: geometry visual box size=0.11 0.02 0.053
